File: hw/oa35-aio/sensors.kicad_sch (KiCad schematic)
At the start: 11 parts, among them U7 ICM-42688-P, U8 BMP280, U9 W25Q128JVSIQ

Commit message: OA35-AIO: placement, autorouting pipeline, production export and docs
- tools/layout.py holds the floorplan: four ESC power blocks in a pinwheel on
  top, flight controller and ESC micros underneath
- tools/gen_pcb.py places the critical parts by hand and the ~150 passives
  automatically, then refuses any overlap or part off the board
- tools/route.py drives freerouting through Specctra DSN/SES and reads the
  session back without needing the KiCad GUI
- tools/finish_pcb.py adds the pours and silkscreen, fills and runs DRC
- tools/export.py writes the JLCPCB gerber zip, BOM and CPL
- docs/ covers the circuit, the Betaflight and AM32 targets, ordering, and
  part substitutions

Co-Authored-By: Claude Opus 5 <noreply@anthropic.com>
Claude-Session: https://claude.ai/code/session_013J1rgXZWykCJN7jVVS67P2
Parts:
- removed R24, R27: 10k, Resistor_SMD:R_0402_1005Metric, symbol oa35:R
- removed R25, R26: 4.7k, Resistor_SMD:R_0402_1005Metric, symbol oa35:R
- added R19, R22: 10k, Resistor_SMD:R_0201_0603Metric, symbol oa35:R
- added R20, R21: 2.4k, Resistor_SMD:R_0201_0603Metric, symbol oa35:R
- C38, C39, C40, C41: footprint Capacitor_SMD:C_0402_1005Metric -> Capacitor_SMD:C_0201_0603Metric; LCSC C1525 -> C181043
Connections:
- net +3V3: now also R19.1, R20.1, R21.1, R22.1
- net FLASH_CS: now also R22.2
- net GYRO_CS: now also R19.2
- net I2C_SCL: now also R20.2
- net I2C_SDA: now also R21.2
Changed lines of the file:
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@@
     (property "Reference" "C38" (at 107.9500 43.7200 0) (effects (font (size 1.27 1.27)) (justify left)))
     (property "Value" "100n" (at 107.9500 50.2600 0) (effects (font (size 1.27 1.27)) (justify left)))
-    (property "Footprint" "Capacitor_SMD:C_0402_1005Metric" (at 110.4900 46.9900 0) (effects (font (size 1.27 1.27)) hide))
+    (property "Footprint" "Capacitor_SMD:C_0201_0603Metric" (at 110.4900 46.9900 0) (effects (font (size 1.27 1.27)) hide))
     (property "Datasheet" "" (at 110.4900 46.9900 0) (effects (font (size 1.27 1.27)) hide))
-    (property "LCSC" "C1525" (at 110.4900 46.9900 0) (effects (font (size 1.27 1.27)) hide))
+    (property "LCSC" "C181043" (at 110.4900 46.9900 0) (effects (font (size 1.27 1.27)) hide))
     (pin "1")
     (pin "2")
@@
     (property "Reference" "C39" (at 165.1000 43.7200 0) (effects (font (size 1.27 1.27)) (justify left)))
     (property "Value" "100n" (at 165.1000 50.2600 0) (effects (font (size 1.27 1.27)) (justify left)))
-    (property "Footprint" "Capacitor_SMD:C_0402_1005Metric" (at 167.6400 46.9900 0) (effects (font (size 1.27 1.27)) hide))
+    (property "Footprint" "Capacitor_SMD:C_0201_0603Metric" (at 167.6400 46.9900 0) (effects (font (size 1.27 1.27)) hide))
     (property "Datasheet" "" (at 167.6400 46.9900 0) (effects (font (size 1.27 1.27)) hide))
-    (property "LCSC" "C1525" (at 167.6400 46.9900 0) (effects (font (size 1.27 1.27)) hide))
+    (property "LCSC" "C181043" (at 167.6400 46.9900 0) (effects (font (size 1.27 1.27)) hide))
     (pin "1")
     (pin "2")
@@
   (symbol (lib_id "oa35:R") (at 224.7900 46.9900 0) (unit 1)
     (in_bom yes) (on_board yes) (dnp no)
-    (property "Reference" "R24" (at 222.2500 43.7200 0) (effects (font (size 1.27 1.27)) (justify left)))
+    (property "Reference" "R19" (at 222.2500 43.7200 0) (effects (font (size 1.27 1.27)) (justify left)))
     (property "Value" "10k" (at 222.2500 50.2600 0) (effects (font (size 1.27 1.27)) (justify left)))
-    (property "Footprint" "Resistor_SMD:R_0402_1005Metric" (at 224.7900 46.9900 0) (effects (font (size 1.27 1.27)) hide))
+    (property "Footprint" "Resistor_SMD:R_0201_0603Metric" (at 224.7900 46.9900 0) (effects (font (size 1.27 1.27)) hide))
     (property "Datasheet" "" (at 224.7900 46.9900 0) (effects (font (size 1.27 1.27)) hide))
-    (property "LCSC" "C25744" (at 224.7900 46.9900 0) (effects (font (size 1.27 1.27)) hide))
+    (property "LCSC" "C106225" (at 224.7900 46.9900 0) (effects (font (size 1.27 1.27)) hide))
     (pin "1")
     (pin "2")
-    (instances (project "oa35-aio" (path "/a68e5d6d-33fe-4995-801f-7fdb090e6968/cfb39ec0-dbc7-4314-80a7-54a974aff431" (reference "R24") (unit 1))))
+    (instances (project "oa35-aio" (path "/a68e5d6d-33fe-4995-801f-7fdb090e6968/cfb39ec0-dbc7-4314-80a7-54a974aff431" (reference "R19") (unit 1))))
   )
   (wire (pts (xy 219.7100 46.9900) (xy 215.9000 46.9900)) (stroke (width 0) (type default)))
@@
     (property "Reference" "C40" (at 50.8000 76.7400 0) (effects (font (size 1.27 1.27)) (justify left)))
     (property "Value" "100n" (at 50.8000 83.2800 0) (effects (font (size 1.27 1.27)) (justify left)))
-    (property "Footprint" "Capacitor_SMD:C_0402_1005Metric" (at 53.3400 80.0100 0) (effects (font (size 1.27 1.27)) hide))
+    (property "Footprint" "Capacitor_SMD:C_0201_0603Metric" (at 53.3400 80.0100 0) (effects (font (size 1.27 1.27)) hide))
     (property "Datasheet" "" (at 53.3400 80.0100 0) (effects (font (size 1.27 1.27)) hide))
-    (property "LCSC" "C1525" (at 53.3400 80.0100 0) (effects (font (size 1.27 1.27)) hide))
+    (property "LCSC" "C181043" (at 53.3400 80.0100 0) (effects (font (size 1.27 1.27)) hide))
     (pin "1")
     (pin "2")
@@
   (symbol (lib_id "oa35:R") (at 110.4900 80.0100 0) (unit 1)
     (in_bom yes) (on_board yes) (dnp no)
-    (property "Reference" "R25" (at 107.9500 76.7400 0) (effects (font (size 1.27 1.27)) (justify left)))
-    (property "Value" "4.7k" (at 107.9500 83.2800 0) (effects (font (size 1.27 1.27)) (justify left)))
-    (property "Footprint" "Resistor_SMD:R_0402_1005Metric" (at 110.4900 80.0100 0) (effects (font (size 1.27 1.27)) hide))
+    (property "Reference" "R20" (at 107.9500 76.7400 0) (effects (font (size 1.27 1.27)) (justify left)))
+    (property "Value" "2.4k" (at 107.9500 83.2800 0) (effects (font (size 1.27 1.27)) (justify left)))
+    (property "Footprint" "Resistor_SMD:R_0201_0603Metric" (at 110.4900 80.0100 0) (effects (font (size 1.27 1.27)) hide))
     (property "Datasheet" "" (at 110.4900 80.0100 0) (effects (font (size 1.27 1.27)) hide))
-    (property "LCSC" "C25900" (at 110.4900 80.0100 0) (effects (font (size 1.27 1.27)) hide))
+    (property "LCSC" "C166281" (at 110.4900 80.0100 0) (effects (font (size 1.27 1.27)) hide))
     (pin "1")
     (pin "2")
-    (instances (project "oa35-aio" (path "/a68e5d6d-33fe-4995-801f-7fdb090e6968/cfb39ec0-dbc7-4314-80a7-54a974aff431" (reference "R25") (unit 1))))
+    (instances (project "oa35-aio" (path "/a68e5d6d-33fe-4995-801f-7fdb090e6968/cfb39ec0-dbc7-4314-80a7-54a974aff431" (reference "R20") (unit 1))))
   )
   (wire (pts (xy 105.4100 80.0100) (xy 101.6000 80.0100)) (stroke (width 0) (type default)))
@@
   (symbol (lib_id "oa35:R") (at 167.6400 80.0100 0) (unit 1)
     (in_bom yes) (on_board yes) (dnp no)
-    (property "Reference" "R26" (at 165.1000 76.7400 0) (effects (font (size 1.27 1.27)) (justify left)))
-    (property "Value" "4.7k" (at 165.1000 83.2800 0) (effects (font (size 1.27 1.27)) (justify left)))
-    (property "Footprint" "Resistor_SMD:R_0402_1005Metric" (at 167.6400 80.0100 0) (effects (font (size 1.27 1.27)) hide))
+    (property "Reference" "R21" (at 165.1000 76.7400 0) (effects (font (size 1.27 1.27)) (justify left)))
+    (property "Value" "2.4k" (at 165.1000 83.2800 0) (effects (font (size 1.27 1.27)) (justify left)))
+    (property "Footprint" "Resistor_SMD:R_0201_0603Metric" (at 167.6400 80.0100 0) (effects (font (size 1.27 1.27)) hide))
     (property "Datasheet" "" (at 167.6400 80.0100 0) (effects (font (size 1.27 1.27)) hide))
-    (property "LCSC" "C25900" (at 167.6400 80.0100 0) (effects (font (size 1.27 1.27)) hide))
+    (property "LCSC" "C166281" (at 167.6400 80.0100 0) (effects (font (size 1.27 1.27)) hide))
     (pin "1")
     (pin "2")
-    (instances (project "oa35-aio" (path "/a68e5d6d-33fe-4995-801f-7fdb090e6968/cfb39ec0-dbc7-4314-80a7-54a974aff431" (reference "R26") (unit 1))))
+    (instances (project "oa35-aio" (path "/a68e5d6d-33fe-4995-801f-7fdb090e6968/cfb39ec0-dbc7-4314-80a7-54a974aff431" (reference "R21") (unit 1))))
   )
   (wire (pts (xy 162.5600 80.0100) (xy 158.7500 80.0100)) (stroke (width 0) (type default)))
@@
     (property "Reference" "C41" (at 279.4000 76.7400 0) (effects (font (size 1.27 1.27)) (justify left)))
     (property "Value" "100n" (at 279.4000 83.2800 0) (effects (font (size 1.27 1.27)) (justify left)))
-    (property "Footprint" "Capacitor_SMD:C_0402_1005Metric" (at 281.9400 80.0100 0) (effects (font (size 1.27 1.27)) hide))
+    (property "Footprint" "Capacitor_SMD:C_0201_0603Metric" (at 281.9400 80.0100 0) (effects (font (size 1.27 1.27)) hide))
     (property "Datasheet" "" (at 281.9400 80.0100 0) (effects (font (size 1.27 1.27)) hide))
-    (property "LCSC" "C1525" (at 281.9400 80.0100 0) (effects (font (size 1.27 1.27)) hide))
+    (property "LCSC" "C181043" (at 281.9400 80.0100 0) (effects (font (size 1.27 1.27)) hide))
     (pin "1")
     (pin "2")
@@
   (symbol (lib_id "oa35:R") (at 53.3400 113.0300 0) (unit 1)
     (in_bom yes) (on_board yes) (dnp no)
-    (property "Reference" "R27" (at 50.8000 109.7600 0) (effects (font (size 1.27 1.27)) (justify left)))
+    (property "Reference" "R22" (at 50.8000 109.7600 0) (effects (font (size 1.27 1.27)) (justify left)))
     (property "Value" "10k" (at 50.8000 116.3000 0) (effects (font (size 1.27 1.27)) (justify left)))
-    (property "Footprint" "Resistor_SMD:R_0402_1005Metric" (at 53.3400 113.0300 0) (effects (font (size 1.27 1.27)) hide))
+    (property "Footprint" "Resistor_SMD:R_0201_0603Metric" (at 53.3400 113.0300 0) (effects (font (size 1.27 1.27)) hide))
     (property "Datasheet" "" (at 53.3400 113.0300 0) (effects (font (size 1.27 1.27)) hide))
-    (property "LCSC" "C25744" (at 53.3400 113.0300 0) (effects (font (size 1.27 1.27)) hide))
+    (property "LCSC" "C106225" (at 53.3400 113.0300 0) (effects (font (size 1.27 1.27)) hide))
     (pin "1")
     (pin "2")
-    (instances (project "oa35-aio" (path "/a68e5d6d-33fe-4995-801f-7fdb090e6968/cfb39ec0-dbc7-4314-80a7-54a974aff431" (reference "R27") (unit 1))))
+    (instances (project "oa35-aio" (path "/a68e5d6d-33fe-4995-801f-7fdb090e6968/cfb39ec0-dbc7-4314-80a7-54a974aff431" (reference "R22") (unit 1))))
   )
   (wire (pts (xy 48.2600 113.0300) (xy 44.4500 113.0300)) (stroke (width 0) (type default)))
