File: hw/oa35-aio/esc2.kicad_sch (KiCad schematic)
At the start: 39 parts, among them J13 M2A, J14 M2B, J15 M2C, U30 AT32F421G8U7, U31 NSG2065Q

Commit message: OA35-AIO: placement, autorouting pipeline, production export and docs
- tools/layout.py holds the floorplan: four ESC power blocks in a pinwheel on
  top, flight controller and ESC micros underneath
- tools/gen_pcb.py places the critical parts by hand and the ~150 passives
  automatically, then refuses any overlap or part off the board
- tools/route.py drives freerouting through Specctra DSN/SES and reads the
  session back without needing the KiCad GUI
- tools/finish_pcb.py adds the pours and silkscreen, fills and runs DRC
- tools/export.py writes the JLCPCB gerber zip, BOM and CPL
- docs/ covers the circuit, the Betaflight and AM32 targets, ordering, and
  part substitutions

Co-Authored-By: Claude Opus 5 <noreply@anthropic.com>
Claude-Session: https://claude.ai/code/session_013J1rgXZWykCJN7jVVS67P2
Parts:
- CRST2, CVCC2, CVDA2, CVDD2: footprint Capacitor_SMD:C_0402_1005Metric -> Capacitor_SMD:C_0201_0603Metric; LCSC C1525 -> C181043
- RBA2, RBB2, RBC2, RBT02, RCA2, RCB2, RCC2, RRST2: footprint Resistor_SMD:R_0402_1005Metric -> Resistor_SMD:R_0201_0603Metric; LCSC C25744 -> C106225
- RGAH2, RGAL2, RGBH2, RGBL2, RGCH2, RGCL2: value 22R -> 15R; footprint Resistor_SMD:R_0402_1005Metric -> Resistor_SMD:R_0201_0603Metric; LCSC C25092 -> C473542
- RNA2, RNB2, RNC2: footprint Resistor_SMD:R_0402_1005Metric -> Resistor_SMD:R_0201_0603Metric; LCSC C11702 -> C270365
- RSIG2: footprint Resistor_SMD:R_0402_1005Metric -> Resistor_SMD:R_0201_0603Metric; LCSC C25091 -> C226468
- RVDA2: footprint Resistor_SMD:R_0402_1005Metric -> Resistor_SMD:R_0201_0603Metric; LCSC C25077 -> C106226
Connections:
- net GAH_2: now also QAH2.4 (G); no longer QAH2.2 (G)
- net GAL_2: now also QAL2.4 (G); no longer QAL2.2 (G)
- net GBH_2: now also QBH2.4 (G); no longer QBH2.2 (G)
- net GBL_2: now also QBL2.4 (G); no longer QBL2.2 (G)
- net GCH_2: now also QCH2.4 (G); no longer QCH2.2 (G)
- net GCL_2: now also QCL2.4 (G); no longer QCL2.2 (G)
- net GND: now also QAL2.2 (S), QAL2.3 (S), QBL2.2 (S), QBL2.3 (S), QCL2.2 (S), QCL2.3 (S)
- net PH_A_2: now also QAH2.2 (S), QAH2.3 (S), QAL2.5 (D); no longer QAL2.3 (D)
- net PH_B_2: now also QBH2.2 (S), QBH2.3 (S), QBL2.5 (D); no longer QBL2.3 (D)
- net PH_C_2: now also QCH2.2 (S), QCH2.3 (S), QCL2.5 (D); no longer QCL2.3 (D)
- net VBAT: now also QAH2.5 (D), QBH2.5 (D), QCH2.5 (D); no longer QAH2.3 (D), QBH2.3 (D), QCH2.3 (D)
- net +9V6 renamed +10V

Commit message: OA35-AIO: fix current-sense input polarity and LDO no-connects
The INA186 in DCK/SC70-6 is 1 REF, 2 GND, 3 VS, 4 IN+, 5 IN-, 6 OUT, per
KiCad's own INA199xxDCK symbol and the OpenESC symbol library. High-side
sensing needs IN+ on the battery side of the shunt; the reference design
wires it the other way round, which would read zero current. Corrected here
and documented.

Also stop tying the LP5912's NC and open-drain power-good pins to rails, and
give the auto-placer "sit next to X" hints so decoupling lands on the pin it
decouples (mean distance 4.6 mm instead of 6.9 mm).

Co-Authored-By: Claude Opus 5 <noreply@anthropic.com>
Claude-Session: https://claude.ai/code/session_013J1rgXZWykCJN7jVVS67P2
Parts:
- J13, J14, J15: footprint oa35:Pad_4.0x3.0mm -> oa35:Pad_2.8x2.0mm
Changed lines of the file:
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@@
     (property "Reference" "J13" (at 405.1300 213.9000 0) (effects (font (size 1.27 1.27)) (justify left)))
     (property "Value" "M2A" (at 405.1300 220.4400 0) (effects (font (size 1.27 1.27)) (justify left)))
-    (property "Footprint" "oa35:Pad_4.0x3.0mm" (at 406.4000 217.1700 0) (effects (font (size 1.27 1.27)) hide))
+    (property "Footprint" "oa35:Pad_2.8x2.0mm" (at 406.4000 217.1700 0) (effects (font (size 1.27 1.27)) hide))
     (property "Datasheet" "" (at 406.4000 217.1700 0) (effects (font (size 1.27 1.27)) hide))
     (property "LCSC" "" (at 406.4000 217.1700 0) (effects (font (size 1.27 1.27)) hide))
@@
     (property "Reference" "J14" (at 455.9300 213.9000 0) (effects (font (size 1.27 1.27)) (justify left)))
     (property "Value" "M2B" (at 455.9300 220.4400 0) (effects (font (size 1.27 1.27)) (justify left)))
-    (property "Footprint" "oa35:Pad_4.0x3.0mm" (at 457.2000 217.1700 0) (effects (font (size 1.27 1.27)) hide))
+    (property "Footprint" "oa35:Pad_2.8x2.0mm" (at 457.2000 217.1700 0) (effects (font (size 1.27 1.27)) hide))
     (property "Datasheet" "" (at 457.2000 217.1700 0) (effects (font (size 1.27 1.27)) hide))
     (property "LCSC" "" (at 457.2000 217.1700 0) (effects (font (size 1.27 1.27)) hide))
@@
     (property "Reference" "J15" (at 49.5300 267.2400 0) (effects (font (size 1.27 1.27)) (justify left)))
     (property "Value" "M2C" (at 49.5300 273.7800 0) (effects (font (size 1.27 1.27)) (justify left)))
-    (property "Footprint" "oa35:Pad_4.0x3.0mm" (at 50.8000 270.5100 0) (effects (font (size 1.27 1.27)) hide))
+    (property "Footprint" "oa35:Pad_2.8x2.0mm" (at 50.8000 270.5100 0) (effects (font (size 1.27 1.27)) hide))
     (property "Datasheet" "" (at 50.8000 270.5100 0) (effects (font (size 1.27 1.27)) hide))
     (property "LCSC" "" (at 50.8000 270.5100 0) (effects (font (size 1.27 1.27)) hide))
