File: hw/oa35-aio/mcu.kicad_sch (KiCad schematic)
At the start: 29 parts, among them Q1 2N7002, U6 STM32F722RET6, Y1 8MHz

Commit message: OA35-AIO: placement, autorouting pipeline, production export and docs
- tools/layout.py holds the floorplan: four ESC power blocks in a pinwheel on
  top, flight controller and ESC micros underneath
- tools/gen_pcb.py places the critical parts by hand and the ~150 passives
  automatically, then refuses any overlap or part off the board
- tools/route.py drives freerouting through Specctra DSN/SES and reads the
  session back without needing the KiCad GUI
- tools/finish_pcb.py adds the pours and silkscreen, fills and runs DRC
- tools/export.py writes the JLCPCB gerber zip, BOM and CPL
- docs/ covers the circuit, the Betaflight and AM32 targets, ordering, and
  part substitutions

Co-Authored-By: Claude Opus 5 <noreply@anthropic.com>
Claude-Session: https://claude.ai/code/session_013J1rgXZWykCJN7jVVS67P2
Parts:
- removed R19: 10k, Resistor_SMD:R_0402_1005Metric, symbol oa35:R
- removed R20: 1k, Resistor_SMD:R_0402_1005Metric, symbol oa35:R
- removed R21, R23: 100R, Resistor_SMD:R_0402_1005Metric, symbol oa35:R
- removed R22: 100k, Resistor_SMD:R_0402_1005Metric, symbol oa35:R
- added R10, R11: 510R, Resistor_SMD:R_0201_0603Metric, symbol oa35:R
- added R12: 100k, Resistor_SMD:R_0201_0603Metric, symbol oa35:R
- added R8: 10k, Resistor_SMD:R_0201_0603Metric, symbol oa35:R
- added R9: 10R, Resistor_SMD:R_0201_0603Metric, symbol oa35:R
- C25, C26, C27, C28, C29, C32, C34, C37: footprint Capacitor_SMD:C_0402_1005Metric -> Capacitor_SMD:C_0201_0603Metric; LCSC C1525 -> C181043
- C30, C31, C33, C35, C36: footprint Capacitor_SMD:C_0402_1005Metric -> Capacitor_SMD:C_0201_0603Metric
- R13: footprint Resistor_SMD:R_0402_1005Metric -> Resistor_SMD:R_0201_0603Metric; LCSC C25744 -> C106225
- R14: value 10R -> 10k; footprint Resistor_SMD:R_0402_1005Metric -> Resistor_SMD:R_0201_0603Metric; LCSC C25077 -> C106225
- R15: value 470R -> 1k; footprint Resistor_SMD:R_0402_1005Metric -> Resistor_SMD:R_0201_0603Metric; LCSC C25117 -> C270365
- R16: value 470R -> 220R; footprint Resistor_SMD:R_0402_1005Metric -> Resistor_SMD:R_0201_0603Metric; LCSC C25117 -> C226468
- R17: footprint Resistor_SMD:R_0402_1005Metric -> Resistor_SMD:R_0201_0603Metric; LCSC C25741 -> C270364
- R18: value 10k -> 220R; footprint Resistor_SMD:R_0402_1005Metric -> Resistor_SMD:R_0201_0603Metric; LCSC C25744 -> C226468
Connections:
- net +3V3: now also R9.1; no longer R14.1
- net +3V3A: now also R9.2; no longer R14.2
- net ADC_RSSI: now also R14.1, R15.2
- net ADC_VBAT: now also R13.1, R12.2; no longer R17.2, R18.1
- net BEEP_G: now also R16.2, R17.1
- net BEEP_GATE: now also R16.1
- net BOOT0: now also R8.1; no longer R13.1
- net GND: now also R14.2, R17.2, R8.2; no longer R18.2
- net LED0: now also R10.2; no longer R15.2
- net LED0_K: now also R10.1; no longer R15.1
- net LED1: now also R11.2; no longer R16.2
- net LED1_K: now also R11.1; no longer R16.1
- net LED_STRIP: now also R18.1
- net PAD_LED: now also R18.2
- net PAD_RSSI: now also R15.1
- net VBAT: now also R12.1; no longer R17.1
Other:
- moved on the sheet: R13, R14, R15, R16, R17, R18

Commit message: OA35-AIO: keep capacitor footprints honest against their LCSC parts
The 4.7 uF, 1 uF and 20 pF capacitors were being emitted on the 0201 land
pattern while their LCSC parts are 0402, so the BOM and the board disagreed
about the physical part. C() now picks the footprint from the value the same
way R() does, and the BOM prints readable values.

Co-Authored-By: Claude Opus 5 <noreply@anthropic.com>
Claude-Session: https://claude.ai/code/session_013J1rgXZWykCJN7jVVS67P2
Parts:
- C30, C31, C33, C35, C36: footprint Capacitor_SMD:C_0201_0603Metric -> Capacitor_SMD:C_0402_1005Metric
Changed lines of the file:
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@@
     (property "Reference" "C30" (at 410.2100 75.4700 0) (effects (font (size 1.27 1.27)) (justify left)))
     (property "Value" "4.7u" (at 410.2100 82.0100 0) (effects (font (size 1.27 1.27)) (justify left)))
-    (property "Footprint" "Capacitor_SMD:C_0201_0603Metric" (at 412.7500 78.7400 0) (effects (font (size 1.27 1.27)) hide))
+    (property "Footprint" "Capacitor_SMD:C_0402_1005Metric" (at 412.7500 78.7400 0) (effects (font (size 1.27 1.27)) hide))
     (property "Datasheet" "" (at 412.7500 78.7400 0) (effects (font (size 1.27 1.27)) hide))
     (property "LCSC" "C23733" (at 412.7500 78.7400 0) (effects (font (size 1.27 1.27)) hide))
@@
     (property "Reference" "C31" (at 469.9000 75.4700 0) (effects (font (size 1.27 1.27)) (justify left)))
     (property "Value" "4.7u" (at 469.9000 82.0100 0) (effects (font (size 1.27 1.27)) (justify left)))
-    (property "Footprint" "Capacitor_SMD:C_0201_0603Metric" (at 472.4400 78.7400 0) (effects (font (size 1.27 1.27)) hide))
+    (property "Footprint" "Capacitor_SMD:C_0402_1005Metric" (at 472.4400 78.7400 0) (effects (font (size 1.27 1.27)) hide))
     (property "Datasheet" "" (at 472.4400 78.7400 0) (effects (font (size 1.27 1.27)) hide))
     (property "LCSC" "C23733" (at 472.4400 78.7400 0) (effects (font (size 1.27 1.27)) hide))
@@
     (property "Reference" "C33" (at 231.1400 171.9900 0) (effects (font (size 1.27 1.27)) (justify left)))
     (property "Value" "1u" (at 231.1400 178.5300 0) (effects (font (size 1.27 1.27)) (justify left)))
-    (property "Footprint" "Capacitor_SMD:C_0201_0603Metric" (at 233.6800 175.2600 0) (effects (font (size 1.27 1.27)) hide))
+    (property "Footprint" "Capacitor_SMD:C_0402_1005Metric" (at 233.6800 175.2600 0) (effects (font (size 1.27 1.27)) hide))
     (property "Datasheet" "" (at 233.6800 175.2600 0) (effects (font (size 1.27 1.27)) hide))
     (property "LCSC" "C52923" (at 233.6800 175.2600 0) (effects (font (size 1.27 1.27)) hide))
@@
     (property "Reference" "C35" (at 410.2100 171.9900 0) (effects (font (size 1.27 1.27)) (justify left)))
     (property "Value" "20p" (at 410.2100 178.5300 0) (effects (font (size 1.27 1.27)) (justify left)))
-    (property "Footprint" "Capacitor_SMD:C_0201_0603Metric" (at 412.7500 175.2600 0) (effects (font (size 1.27 1.27)) hide))
+    (property "Footprint" "Capacitor_SMD:C_0402_1005Metric" (at 412.7500 175.2600 0) (effects (font (size 1.27 1.27)) hide))
     (property "Datasheet" "" (at 412.7500 175.2600 0) (effects (font (size 1.27 1.27)) hide))
     (property "LCSC" "C1554" (at 412.7500 175.2600 0) (effects (font (size 1.27 1.27)) hide))
@@
     (property "Reference" "C36" (at 469.9000 171.9900 0) (effects (font (size 1.27 1.27)) (justify left)))
     (property "Value" "20p" (at 469.9000 178.5300 0) (effects (font (size 1.27 1.27)) (justify left)))
-    (property "Footprint" "Capacitor_SMD:C_0201_0603Metric" (at 472.4400 175.2600 0) (effects (font (size 1.27 1.27)) hide))
+    (property "Footprint" "Capacitor_SMD:C_0402_1005Metric" (at 472.4400 175.2600 0) (effects (font (size 1.27 1.27)) hide))
     (property "Datasheet" "" (at 472.4400 175.2600 0) (effects (font (size 1.27 1.27)) hide))
     (property "LCSC" "C1554" (at 472.4400 175.2600 0) (effects (font (size 1.27 1.27)) hide))
