File: hw/oa35-aio/power.kicad_sch (KiCad schematic)
At the start: 53 parts, among them J3 BAT+, J4 BAT-, J5 CAP+, J6 CAP-, U1 INA186A3IDCKR, U2 LMR51430YFDDCR, U3 LMR51430YFDDCR, U4 LP5912-3.3DRVR, U5 TLV76733DRVR

Commit message: OA35-AIO: placement, autorouting pipeline, production export and docs
- tools/layout.py holds the floorplan: four ESC power blocks in a pinwheel on
  top, flight controller and ESC micros underneath
- tools/gen_pcb.py places the critical parts by hand and the ~150 passives
  automatically, then refuses any overlap or part off the board
- tools/route.py drives freerouting through Specctra DSN/SES and reads the
  session back without needing the KiCad GUI
- tools/finish_pcb.py adds the pours and silkscreen, fills and runs DRC
- tools/export.py writes the JLCPCB gerber zip, BOM and CPL
- docs/ covers the circuit, the Betaflight and AM32 targets, ordering, and
  part substitutions

Co-Authored-By: Claude Opus 5 <noreply@anthropic.com>
Claude-Session: https://claude.ai/code/session_013J1rgXZWykCJN7jVVS67P2
Parts:
- removed R11, R12: 2.4k, Resistor_SMD:R_0402_1005Metric, symbol oa35:R
- removed R8: 1k, Resistor_SMD:R_0402_1005Metric, symbol oa35:R
- C11, C12, C15, C17, C18, C20, C21, C22, C24, C6, C7, C8: footprint Capacitor_SMD:C_0402_1005Metric -> Capacitor_SMD:C_0201_0603Metric; LCSC C1525 -> C181043
- C19, C23: footprint Capacitor_SMD:C_0402_1005Metric -> Capacitor_SMD:C_0201_0603Metric
- R1: footprint Resistor_SMD:R_0402_1005Metric -> Resistor_SMD:R_0201_0603Metric; LCSC C11702 -> C270365
- R2: footprint Resistor_SMD:R_0402_1005Metric -> Resistor_SMD:R_0201_0603Metric; LCSC C25741 -> C270364
- R3: value 10k -> 6.49k; footprint Resistor_SMD:R_0402_1005Metric -> Resistor_SMD:R_0201_0603Metric; LCSC C25744 -> C2107920
- R4: value 20k -> 100k; footprint Resistor_SMD:R_0402_1005Metric -> Resistor_SMD:R_0201_0603Metric; LCSC C25765 -> C270364
- R5: value 100k -> 13.7k; footprint Resistor_SMD:R_0402_1005Metric -> Resistor_SMD:R_0201_0603Metric; LCSC C25741 -> C320695
- R6: value 10k -> 2.4k; footprint Resistor_SMD:R_0402_1005Metric -> Resistor_SMD:R_0201_0603Metric; LCSC C25744 -> C166281
- R7: footprint Resistor_SMD:R_0402_1005Metric -> Resistor_SMD:R_0201_0603Metric; LCSC C25882 -> C166281
Connections:
- net FB_5Vb is gone; now on net +3V3_LED: R7.2
- net +3V3: now also R7.1
- net +5V: now also R6.1
- net +5V_BUCK: now also R4.1; no longer R5.1
- net +5V_LED: now also R6.2
- net FB_5V: now also R4.2, R5.1; no longer R5.2, R6.1
- net FB_GD: no longer R4.1
- net GND: now also R5.2; no longer R4.2
- net +9V6 renamed +10V
- removed net FB_5Va: R6.2, R7.1
Other:
- moved on the sheet: C10, C11, C12, C13, C14, C15, C16, C17, C18, C19, C20, C21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

Commit message: OA35-AIO: fix current-sense input polarity and LDO no-connects
The INA186 in DCK/SC70-6 is 1 REF, 2 GND, 3 VS, 4 IN+, 5 IN-, 6 OUT, per
KiCad's own INA199xxDCK symbol and the OpenESC symbol library. High-side
sensing needs IN+ on the battery side of the shunt; the reference design
wires it the other way round, which would read zero current. Corrected here
and documented.

Also stop tying the LP5912's NC and open-drain power-good pins to rails, and
give the auto-placer "sit next to X" hints so decoupling lands on the pin it
decouples (mean distance 4.6 mm instead of 6.9 mm).

Co-Authored-By: Claude Opus 5 <noreply@anthropic.com>
Claude-Session: https://claude.ai/code/session_013J1rgXZWykCJN7jVVS67P2
Parts:
- removed J5: CAP+, oa35:Pad_4.0x3.0mm, symbol oa35:PAD
- removed J6: CAP-, oa35:Pad_4.0x3.0mm, symbol oa35:PAD
Connections:
- net +3V3: no longer U4.2 (OUT)
- net GND: no longer U4.5 (EN)
- net VBAT: now also U1.5 (IN-); no longer U1.4 (IN-)
- net VBAT_IN: now also U1.4 (IN+); no longer U1.5 (IN+)
- no-connect marks 0 -> 2
Other:
- moved on the sheet: C1, C10, C11, C12, C13, C14, C15, C16, C17, C18, C19, C2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

Commit message: OA35-AIO: keep capacitor footprints honest against their LCSC parts
The 4.7 uF, 1 uF and 20 pF capacitors were being emitted on the 0201 land
pattern while their LCSC parts are 0402, so the BOM and the board disagreed
about the physical part. C() now picks the footprint from the value the same
way R() does, and the BOM prints readable values.

Co-Authored-By: Claude Opus 5 <noreply@anthropic.com>
Claude-Session: https://claude.ai/code/session_013J1rgXZWykCJN7jVVS67P2
Parts:
- C19, C23: footprint Capacitor_SMD:C_0201_0603Metric -> Capacitor_SMD:C_0402_1005Metric
Changed lines of the file:
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@@
     (property "Reference" "C19" (at 403.8600 116.1100 0) (effects (font (size 1.27 1.27)) (justify left)))
     (property "Value" "4.7u" (at 403.8600 122.6500 0) (effects (font (size 1.27 1.27)) (justify left)))
-    (property "Footprint" "Capacitor_SMD:C_0201_0603Metric" (at 406.4000 119.3800 0) (effects (font (size 1.27 1.27)) hide))
+    (property "Footprint" "Capacitor_SMD:C_0402_1005Metric" (at 406.4000 119.3800 0) (effects (font (size 1.27 1.27)) hide))
     (property "Datasheet" "" (at 406.4000 119.3800 0) (effects (font (size 1.27 1.27)) hide))
     (property "LCSC" "C23733" (at 406.4000 119.3800 0) (effects (font (size 1.27 1.27)) hide))
@@
     (property "Reference" "C23" (at 149.8600 141.5100 0) (effects (font (size 1.27 1.27)) (justify left)))
     (property "Value" "4.7u" (at 149.8600 148.0500 0) (effects (font (size 1.27 1.27)) (justify left)))
-    (property "Footprint" "Capacitor_SMD:C_0201_0603Metric" (at 152.4000 144.7800 0) (effects (font (size 1.27 1.27)) hide))
+    (property "Footprint" "Capacitor_SMD:C_0402_1005Metric" (at 152.4000 144.7800 0) (effects (font (size 1.27 1.27)) hide))
     (property "Datasheet" "" (at 152.4000 144.7800 0) (effects (font (size 1.27 1.27)) hide))
     (property "LCSC" "C23733" (at 152.4000 144.7800 0) (effects (font (size 1.27 1.27)) hide))
